File: LSwarm Anchor PCB/LSwarm Anchor PCB.kicad_pcb (KiCad board)
At the start: 4 copper layers, 94.5 x 31 mm, 59 parts, among them Q7 AO3407A, SW1 MSK12C02, U1 BQ24075RGTR, U12 AP2112K-3.3, U2 BU03, U4 DW03C_C41367942, U6 ESP32-C3-MINI-1U-N4

Commit message: sync
Parts:
- removed D4, D7, D8: LED, LED_SMD:LED_0402_1005Metric
- added LED4: KT-0603R, easyeda2kicad:LED-SMD_L1.6-W0.8-R-RD, F.Cu at (36.8, 1.75)
- added LED5: KT-0603R, easyeda2kicad:LED-SMD_L1.6-W0.8-R-RD, F.Cu at (22.8, 1.75)
- added LED6: KT-0603R, easyeda2kicad:LED-SMD_L1.6-W0.8-R-RD, F.Cu at (27.5, 1.75)
- moved G*** 20.1 mm to (44.8, 7.00), turned to 180 degrees
- moved R29 1.87 mm to (22.8, 3.75)
- moved R24 1.03 mm to (27.6, 3.75)
- moved R21 0.75 mm to (36.6, 3.75)
Routing:
- net Net-(LED5-K): track 25.0 -> 22.9 mm
- net Net-(LED6-K): track 26.2 -> 27.3 mm
