File: LSwarm Anchor PCB/LSwarm Anchor PCB.kicad_sch (KiCad schematic)
At the start: 0 parts

Commit message: sync
Parts:
- added BT1: BH-18650-A1AJ006, easyeda2kicad:BAT-TH_BH-18650-A1AJ006, symbol easyeda2kicad:BH-18650-A1AJ006
- added BUZZER2: MLT-5020, easyeda2kicad:BUZ-SMD_L5.0-W5.5-P4.60, symbol easyeda2kicad:MLT-5020
- added C1: CL21A226MAQNNNE, easyeda2kicad:C0805, symbol easyeda2kicad:CL21A226MAQNNNE
- added C27: 10nF, Capacitor_SMD:C_0603_1608Metric, symbol Device:C
- added C31, C32, C41, C52, C65: 1uF, Capacitor_SMD:C_0603_1608Metric, symbol Device:C
- added C40, C55, C62: 10uF, Capacitor_SMD:C_0603_1608Metric, symbol Device:C
- added C56, C58, C59, C61: 100nf, Capacitor_SMD:C_0603_1608Metric, symbol Device:C
- added C71: 100nF, Capacitor_SMD:C_0603_1608Metric, symbol Device:C
- added C71C1: 10uF, Capacitor_SMD:C_0805_2012Metric, symbol Device:C
- added D4, D7, D8: LED, LED_SMD:LED_0402_1005Metric, symbol Device:LED
- added D5: USBLC6-2SC6_C2687116, easyeda2kicad:SOT-23-6_L2.9-W1.6-P0.95-LS2.8-BL, symbol easyeda2kicad:USBLC6-2SC6_C2687116
- added L1: MPZ2012S601AT000, easyeda2kicad:L0805, symbol easyeda2kicad:MPZ2012S601AT000
- added Q7: AO3407A, easyeda2kicad:SOT-23-3_L2.9-W1.6-P1.90-LS2.8-BR, symbol easyeda2kicad:AO3407A
- added R11: 1.5k, Resistor_SMD:R_0603_1608Metric, symbol Device:R
- added R12, R18, R23, R32, R33, R39: 10k, Resistor_SMD:R_0603_1608Metric, symbol Device:R
- added R16: 470, Resistor_SMD:R_0603_1608Metric, symbol Device:R
- added R21, R24, R29, R9: 1k, Resistor_SMD:R_0603_1608Metric, symbol Device:R
- added R25, R26: 220k, Resistor_SMD:R_0603_1608Metric, symbol Device:R
- added R27: 100, Resistor_SMD:R_0603_1608Metric, symbol Device:R
- added R28, R40: 100k, Resistor_SMD:R_0603_1608Metric, symbol Device:R
- added R34, R37: 5.1k, Resistor_SMD:R_0603_1608Metric, symbol Device:R
- added R35, R36: 27, Resistor_SMD:R_0603_1608Metric, symbol Device:R
- added SW1: MSK12C02, easyeda2kicad:SW-TH_MSK12C02, symbol easyeda2kicad:MSK12C02
- added TP34: ESP32_EN, TestPoint:TestPoint_Pad_1.0x1.0mm, symbol Connector:TestPoint
- added TP36: ESP32_BOOT, TestPoint:TestPoint_Pad_1.0x1.0mm, symbol Connector:TestPoint
- added TP38: ESP32_RX, TestPoint:TestPoint_Pad_1.0x1.0mm, symbol Connector:TestPoint
- added TP40: ESP32_TX, TestPoint:TestPoint_Pad_1.0x1.0mm, symbol Connector:TestPoint
- added U1: BQ24075RGTR, easyeda2kicad:QFN-16_L3.0-W3.0-P0.50-TL-EP1.7, symbol easyeda2kicad:BQ24075RGTR
- added U12: AP2112K-3.3, Package_TO_SOT_SMD:SOT-23-5, symbol Regulator_Linear:AP2112K-3.3
- added U2: BU03, easyeda2kicad:WIRELM-SMD_BU03, symbol easyeda2kicad:BU03
- added U4: DW03C_C41367942, easyeda2kicad:SOT-23-5_L2.9-W1.6-P0.95-LS2.9-BL, symbol easyeda2kicad:DW03C_C41367942
- added U6: ESP32-C3-MINI-1U-N4, easyeda2kicad:WIFIM-SMD_61P-L13.2-W12.5-P0.80, symbol easyeda2kicad:ESP32-C3-MINI-1U-N4
- added USB1: USB-TYPE-C-018, easyeda2kicad:USB-C_SMD-TYPE-C-31-M-12, symbol easyeda2kicad:USB-TYPE-C-018
Connections:
- new net: C31.1, R16.2, U4.3 (VDD)
- new net: C56.1, U6.3 (3V3)
- new net: C55.1, C56.2
- new net: C52.2, R18.1, TP34.1, U6.8 (EN)
- new net: D7.2 (A), R24.2
- new net: Q7.1 (G), R23.2, R28.1
- new net: D8.1 (K), U1.7 (#PGOOD)
- new net: D8.2 (A), R29.2
- new net: R11.1, U1.12 (ILIM)
- new net: C27.2, USB1.0 (SH), USB1.1 (SH), USB1.2 (SH), USB1.3 (SH)
- new net: D7.1 (K), U1.9 (#CHG)
- new net: BUZZER2.1 (+), R27.2
- new net: C40.2, C41.2
- new net: R23.1, SW1.2
- new net: D5.4 (I/O2), R36.2
- new net: D5.6 (I/O1), R35.1
- new net: R12.1, U1.1 (TS)
- new net: R9.1, U1.16 (ISET)
- new net: TP38.1, U6.30 (RXD0)
- new net: R34.2, USB1.B5 (CC2)
- new net: D4.2 (A), R21.2
- new net: TP40.1, U6.31 (TXD0)
- new net: R37.1, USB1.A5 (CC1)
- new net: TP36.1, U6.23 (IO9)
- new net +3.3V: C55.2, L1.2, R18.2, R21.1, R24.1, R29.1, R32.1, R33.1, R39.1, U12.5 (VOUT)
- new net BATT+: BT1.2, R16.1, R25.1, U1.2 (BAT), U1.3 (BAT)
- new net BATT-: BT1.1, U4.2 (GND)
- new net BATT_OUT: C40.1, Q7.2 (S), R28.2, U1.10 (OUT), U1.11 (OUT), U1.5 (EN2)
- new net BATT_SW+: C1.1, C65.2, C71C1.2, Q7.3 (D), U12.1 (VIN), U12.3 (EN)
- new net DW_CLK: U2.20 (CLK), U6.20 (IO6)
- new net DW_IRQ: R40.2, U2.22 (IRQ), U6.6 (IO3)
- new net DW_MISO: U2.19 (MISO), U6.18 (IO4)
- new net DW_MOSI: U2.18 (MOSI), U6.19 (IO5)
- new net DW_RST: U2.3 (RSTN), U6.16 (IO10)
- new net DW_Sn: R39.2, U2.17 (CSN), U6.21 (IO7)
- new net DW_WAKEUP: U2.2 (WAKEUP), U6.13 (IO1)
- new net ESP32_BUZZ: R27.1, R33.2, U6.22 (IO8)
- new net ESP32_STATUS: D4.1 (K), R32.2, U6.5 (IO2)
- new net ESP32_USB_DN: R35.2, U6.26 (IO18)
- new net ESP32_USB_DP: R36.1, U6.27 (IO19)
- new net ESP32_VMON_ADC: C71.2, R25.2, R26.2, U6.12 (IO0)
- new net GND: BUZZER2.2 (-), C1.2, C27.1, C31.2, C32.1, C41.1, C52.1, C58.2, C59.2, C61.2, C62.2, C65.1, C71.1, C71C1.1, D5.2 (GND), R11.2, R12.2, R26.1, R34.1, R37.2, R40.1, R9.2, SW1.3, U1.15 (SYSOFF), U1.17 (EP), U1.4 (#CE), U1.6 (EN1), U1.8 (VSS), U12.2 (GND), U2.16 (GND), U2.24 (GND), U2.8 (GND), U4.4 (VM), U6.1 (GND), U6.11 (GND), U6.14 (GND), U6.2 (GND), U6.36 (GND), U6.37 (GND), U6.38 (GND), U6.39 (GND), U6.40 (GND), U6.41 (GND), U6.42 (GND), U6.43 (GND), U6.44 (GND), U6.45 (GND), U6.46 (GND), U6.47 (GND), U6.48 (GND), U6.49 (GND), U6.50 (GND), U6.51 (GND), U6.52 (GND), U6.53 (GND), U6.54 (GND), U6.55 (GND), U6.56 (GND), U6.57 (GND), U6.58 (GND), U6.59 (GND), U6.60 (GND), U6.61 (GND), USB1.A1 (GND), USB1.A12 (GND), USB1.B1 (GND), USB1.B12 (GND)
- new net USB_D+: D5.3 (I/O2), USB1.A6 (DP1), USB1.B6 (DP2)
- new net USB_D-: D5.1 (I/O1), USB1.A7 (DN1), USB1.B7 (DN2)
- new net USB_VBUS: C32.2, D5.5 (VBUS), U1.13 (IN), USB1.A4 (VBUS), USB1.A9 (VBUS), USB1.B4 (VBUS), USB1.B9 (VBUS)
- new net UW_3.3V: C58.1, C59.1, C61.1, C62.1, L1.1, U2.5 (VDD), U2.6 (VCC), U2.7 (VCC)
- no-connect marks 0 -> 33
Other:
- note added: "3.3V REG"
- note added: "ARM"
- note added: "BUZZ"
- note added: "Batt Connector"
- note added: "Batt Protection"
- note added: "Charger"
- note added: "ESD Protection"
- note added: "ESP32"
- note added: "STATUS"
- note added: "USB-C Connector"
- note added: "UWB ANCHOR"
- note added: "V MON"

Commit message: sync
Parts:
- added TP39: 3.3V REF, TestPoint:TestPoint_Pad_1.0x1.0mm, symbol Connector:TestPoint
- added TP41: GND REF, TestPoint:TestPoint_Pad_1.0x1.0mm, symbol Connector:TestPoint
Connections:
- net +3.3V: now also TP39.1
- net GND: now also TP41.1

Commit message: sync
Parts:
- removed D4, D7, D8: LED, LED_SMD:LED_0402_1005Metric, symbol Device:LED
- added LED4, LED5, LED6: KT-0603R, easyeda2kicad:LED-SMD_L1.6-W0.8-R-RD, symbol easyeda2kicad:KT-0603R
Connections:
- net ESP32_STATUS: now also LED4.2 (K)
- net at R24.2: now also LED6.1 (A)
- net at U1.7 (#PGOOD): now also LED5.2 (K)
- net at R29.2: now also LED5.1 (A)
- net at U1.9 (#CHG): now also LED6.2 (K)
- net at R21.2: now also LED4.1 (A)
Other:
- moved on the sheet: R24, R29
